File: Snap_Station.kicad_sch (KiCad schematic)
At the start: 125 parts, among them J11 Printer Problem Lamp, J12 Barrel_Jack_Near_Card_Reader, J13 Print Button, J14 Remove Cartridge Button, J15 N64 Interface Board, J16 Coincard Interface, J2 N64 AC Power Relay, J3 To N64 Port #4, J4 Video Printer, J6 Barrel_Jack_Near_PIC, J8 Paper Sensor, P1 Card Reader, Q1 NDS355AN, Q2 NDS355AN, U1 74HC595, U10 LM7805_TO220, U11 MAX232, U13 74HCT02D, U3 2 MHz Resonator, U4 PIC16C65A-20_P, U5 CNT-NUS, U6 74HCT30D,652, U7 74HCT02D, Y1 Crystal

Commit message: Add files via upload
Connections:
- net CNT-NUS.E12 renamed D0
- net CNT-NUS.E13 renamed D1
- net CNT-NUS.E16 renamed D2
- net CNT-NUS.E2 renamed A14
- net CNT-NUS.E2.Output renamed A14.Inverted
- net CNT-NUS.E20 renamed WE
- net CNT-NUS.E25 renamed A0-A4-OE
- net CNT-NUS.E27 renamed D7
- net CNT-NUS.E28 renamed D6
- net CNT-NUS.E29 renamed D5
- net CNT-NUS.E30 renamed D4
- net CNT-NUS.E32 renamed D3
- net HCT30-E20.Output renamed A0-A4-WE
Other:
- moved on the sheet: R34, R36, R37, R38, R39, R40
